Commit message: 1028_1629_调整了H1_2的URDF

File: source/whole_body_tracking/whole_body_tracking/assets/unitree_h1_2/h1_2.urdf (robot description, URDF)
Before this commit: robot h1_2, 58 links, 57 joints
Joints:
- joint left_shoulder_roll_joint: parent left_shoulder_pitch_link -> left_shoulder_pitc h_link
